File: hardware/kicad/AutoMate_Custom_PCB/AutoMate.kicad_pcb (KiCad board)
At the start: 8 copper layers, 71 parts, among them J1 8P8C, J11_Doorsensor1 Conn_01x02_Socket, J12_ZMCT103C1 Conn_01x02_Socket, J2_BH1750 Conn_01x05_Socket, J2_IR_AHT_BH17 Conn_01x05_Socket, J2_IR_AHT_BH18 Conn_01x05_Socket, J2_PCA9685_Female1 PCA9685, J2_PCA9685_Male1 PCA9685, J5_Relay1 Relay, J9_AHT_BMP1 Conn_01x04_Socket, J9_ZMPT1 Conn_01x04_Socket, SW1_Manual_Override1 SW_DIP_x12, T1 Screw_Terminal_01x02, T10 ST01x02, T11 ST01x02, T12 ST01x02, T13 ST01x02, T14 ST01x02, T15 ST01x02, T2 Screw_Terminal_01x02, T3 Screw_Terminal_01x02, T4 Screw_Terminal_01x02, T5 Screw_Terminal_01x02, T6 Screw_Terminal_01x02, T7 Screw_Terminal_01x02, T8 ST01x02, T9 ST01x02, U1 815, U1_ESP32-DEVKITC1 ESP32-DEVKITC, U2_74HC595 74HC595

Commit message: v1.0.3: Fix 12V driver automation and state persistence
Parts:
- J2_PCA9685_Female1: footprint Connector_PinHeader_2.54mm:PinHeader_1x06_P2.54mm_Horizontal -> Connector_PinSocket_2.54mm:PinSocket_1x06_P2.54mm_Horizontal
- moved J2_PCA9685_Female1 12.7 mm to (101.6, 124.5), turned to 180 degrees
- moved AC1_ACinput1 2.54 mm to (58.4, 152.4)
- moved U2_74HC595 2.54 mm to (35.6, 147.3)
Connections:
- J2_PCA9685_Female1 pad 1: GND -> unconnected-(J2_PCA9685_Female1-Pin_1-Pad1)
- J2_PCA9685_Female1 pad 2: unconnected-(J2_PCA9685_Female1-Pin_2-Pad2) -> +5V
- J2_PCA9685_Female1 pad 3: I2C_SCL -> I2C_SDA
- J2_PCA9685_Female1 pad 4: I2C_SDA -> I2C_SCL
- J2_PCA9685_Female1 pad 5: +5V -> unconnected-(J2_PCA9685_Female1-Pin_5-Pad5)
- J2_PCA9685_Female1 pad 6: unconnected-(J2_PCA9685_Female1-Pin_6-Pad6) -> GND
Routing:
- net GND: track 721.7 -> 728.7 mm
- net Net-(U2_74HC595-QH): track 5.08 -> 0.00 mm
- net Net-(U2_74HC595-QG): track 5.08 -> 0.00 mm
- net Net-(U2_74HC595-QF): track 5.08 -> 0.00 mm
- net Net-(U2_74HC595-QE): track 5.08 -> 0.00 mm
- net Net-(U2_74HC595-QD): track 5.08 -> 0.00 mm
- net Net-(U2_74HC595-QC): track 5.08 -> 0.00 mm
- net Net-(U2_74HC595-QB): track 5.08 -> 0.00 mm
- net +3.3V: track 81.0 -> 84.6 mm
- net SER: track 9.72 -> 12.3 mm
- net Net-(U2_74HC595-QA): track 14.8 -> 12.3 mm
- net SRCLK: track 31.1 -> 33.3 mm
- net RCLK: track 9.72 -> 11.9 mm
- net Net-(U2_74HC595-~{SRCLR}): track 21.4 -> 22.4 mm
